Commit message: - mirobot task no error

File: assets/urdf/mirobot_description/mirobot.urdf (robot description, URDF)
Before this commit: robot mirobot_urdf_2, 10 links, 9 joints
Links:
- link Link1: geometry collision mesh filename=assets/urdf/mirobot_description/meshes/Link1.obj; visual mesh filename=assets/urdf/mirobot_description/meshes/Link1.dae
- link Link2: geometry collision mesh filename=assets/urdf/mirobot_description/meshes/Link2.obj; visual mesh filename=assets/urdf/mirobot_description/meshes/Link2.dae
- link Link3: geometry collision mesh filename=assets/urdf/mirobot_description/meshes/Link3.obj; visual mesh filename=assets/urdf/mirobot_description/meshes/Link3.dae
- link Link4: geometry collision mesh filename=assets/urdf/mirobot_description/meshes/Link4.obj; visual mesh filename=assets/urdf/mirobot_description/meshes/Link4.dae
- link Link5: geometry collision mesh filename=assets/urdf/mirobot_description/meshes/Link5_align.obj; visual mesh filename=assets/urdf/mirobot_description/meshes/Link5_align.dae
- link Link6: geometry collision mesh filename=assets/urdf/mirobot_description/meshes/Link6.obj; visual mesh filename=assets/urdf/mirobot_description/meshes/Link6.dae
- link base_link: geometry collision mesh filename=assets/urdf/mirobot_description/meshes/base_link.obj; visual mesh filename=assets/urdf/mirobot_description/meshes/base_link.dae
- link left_finger: geometry collision mesh filename=assets/urdf/mirobot_description/meshes/mirobot_leftfinger.o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; visual mesh filename=assets/urdf/mirobot_description/meshes/mirobot_leftfinger.o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
- link mirobot_hand: geometry collision mesh filename=assets/urdf/mirobot_description/meshes/mirobot_hand.obj; visual mesh filename=assets/urdf/mirobot_description/meshes/mirobot_hand.obj
- link right_finger: geometry collision mesh filename=assets/urdf/mirobot_description/meshes/mirobot_rightfinger.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; visual mesh filename=assets/urdf/mirobot_description/meshes/mirobot_rightfinger.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

File: assets/urdf/objects/cube_multicolor.urdf (robot description, URDF)
Before this commit: robot object, 1 links, 0 joints
Links:
- removed link object
- added link cube; collision box size=0.05 0.05 0.05; visual mesh filename=meshes/cube_multicolor.obj scale=.05 .05 .05

Commit message: - cube approach rl success

File: assets/urdf/mirobot_description/mirobot.urdf (robot description, URDF)
Before this commit: robot mirobot_urdf_2, 10 links, 9 joints
Joints:
- joint joint1: limit lower=-1.7453 upper=2.7925 effort=80 velocity=1.1344 -> lower=-1.7453 upper=1.7453 effort=80 velocity=1.1344
- joint joint2: limit lower=-0.5235 upper=1.2217 effort=50 velocity=1.1344 -> lower=-1.0471 upper=1.5707 effort=50 velocity=1.1344
- joint joint3: limit lower=-2.967 upper=1.0471 effort=10 velocity=0.4886 -> lower=-3.1415 upper=0.8726 effort=10 velocity=0.4886
- joint joint4: limit lower=-6.1086 upper=6.1086 effort=10 velocity=1.9198 -> lower=-3.1415 upper=3.1415 effort=10 velocity=1.9198
- joint joint5: limit lower=-3.5779 upper=0.6283 effort=10 velocity=0.5759 -> lower=-3.14 upper=0.698 effort=10 velocity=0.5759

Commit message: - mirobot material setting

File: assets/urdf/mirobot_description/mirobot.urdf (robot description, URDF)
Before this commit: robot mirobot_urdf_2, 10 links, 9 joints
Links:
- link left_finger: geometry collision mesh filename=assets/urdf/mirobot_description/meshes/mirobot_leftfinger.o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; visual mesh filename=assets/urdf/mirobot_description/meshes/mirobot_leftfinger.d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
- link mirobot_hand: geometry collision mesh filename=assets/urdf/mirobot_description/meshes/mirobot_hand.obj; visual mesh filename=assets/urdf/mirobot_description/meshes/mirobot_hand.dae
