Commit message: - robotiq 85 gripper sync and limit bug fix

File: assets/urdf/objects/paper_cup.urdf (robot description, URDF)
Before this commit: robot paper_cup, 1 links, 0 joints
Links:
- link paper_cup: geometry collision mesh filename=package://objects/meshes/paper_cup.obj scale=1 1 1; visual mesh filename=package://objects/meshes/paper_cup.obj scale=1 1 1

File: assets/urdf/ur3_description/robot/ur3_robotiq85_gripper.urdf (robot description, URDF)
Before this commit: robot ur5, 21 links, 20 joints
Joints:
- joint robotiq_85_left_finger_tip_joint: limit lower=-3.14 upper=3.14 effort=1000 velocity=1.0 -> lower=-0.80285 upper=0.0 effort=100 velocity=0.2; mimic joint=robotiq_85_left_knuckle_joint multiplier=-1 -> (none); type continuous -> revolute
- joint robotiq_85_left_inner_knuckle_joint: limit lower=-3.14 upper=3.14 effort=1000 velocity=1.0 -> lower=0.0 upper=0.80285 effort=100 velocity=0.2; mimic joint=robotiq_85_left_knuckle_joint offset=0 -> (none); type continuous -> revolute
- joint robotiq_85_left_knuckle_joint: limit lower=0.0 upper=0.80285 effort=1000 velocity=0.5 -> lower=0.0 upper=0.80285 effort=100 velocity=0.2
- joint robotiq_85_right_finger_tip_joint: limit lower=-3.14 upper=3.14 effort=1000 velocity=1.0 -> lower=-0.80285 upper=0.0 effort=100 velocity=0.2; mimic joint=robotiq_85_left_knuckle_joint multiplier=-1 -> (none); type continuous -> revolute
- joint robotiq_85_right_inner_knuckle_joint: limit lower=-3.14 upper=3.14 effort=1000 velocity=1.0 -> lower=0.0 upper=0.80285 effort=100 velocity=0.2; mimic joint=robotiq_85_left_knuckle_joint offset=0 -> (none); type continuous -> revolute
- joint robotiq_85_right_knuckle_joint: limit lower=-3.14 upper=3.14 effort=1000 velocity=0.5 -> lower=0.0 upper=0.80285 effort=100 velocity=0.2; mimic joint=robotiq_85_left_knuckle_joint -> (none); type continuous -> revolute
