Commit message: - naming change from mirobot to ur3 - reset code update - bug fix. - bottle respawn

File: assets/urdf/objects/bottle.urdf (robot description, URDF)
Before this commit: robot paper_cup, 1 links, 0 joints
Links:
- link paper_cup: geometry collision mesh filename=package://objects/meshes/bottle_collision.obj scale=1 1 1; visual mesh filename=package://objects/meshes/bottle.obj scale=1 1 1

Commit message: - grasping & lifting skill learning success with cup object - target objects' physical properties are corrected

File: assets/urdf/objects/bottle.urdf (robot description, URDF)
Before this commit: robot paper_cup, 1 links, 0 joints
Links:
- removed link paper_cup
- added link bottle, mass 0.109; collision mesh filename=package://objects/meshes/bottle.obj scale=1 1 1; visual mesh filename=package://objects/meshes/bottle.obj scale=1 1 1

File: assets/urdf/objects/paper_cup.urdf (robot description, URDF)
Before this commit: robot paper_cup, 1 links, 0 joints
Links:
- link paper_cup: mass 0.00408 -> 0.014

Commit message: - add bottle model with more thick floor - add liquid sphere model - reward shaping including the liquid

File: assets/urdf/objects/bottle.urdf (robot description, URDF)
Before this commit: robot bottle, 1 links, 0 joints
Links:
- link bottle: geometry collision mesh filename=package://objects/meshes/bottle2.obj scale=1 1 1; visual mesh filename=package://objects/meshes/bottle2.obj scale=1 1 1
