Commit message: - gourd_bottle bug fixed

File: assets/urdf/objects/gourd_bottle.urdf (robot description, URDF)
Before this commit: robot gourd_bottle, 1 links, 0 joints
Links:
- removed link gourd_bottle
- added link bottle, mass 0.2; collision mesh filename=package://objects/meshes/gourd_bottle.obj scale=1 1 1; visual mesh filename=package://objects/meshes/gourd_bottle.obj scale=1 1 1
