Commit message: - bottle collision shape change to octagonal shape - solve(rel) function check finish - reset target error fix! - learning grasping bottle skill in task space

File: assets/urdf/ur3_description/robot/ur3_robotiq85_gripper.urdf (robot description, URDF)
Before this commit: robot ur5, 21 links, 20 joints
Joints:
- joint robotiq_85_left_finger_tip_joint: limit lower=-3.14 upper=3.14 effort=0.1 velocity=100.0 -> lower=-3.14 upper=3.14 effort=1000 velocity=1.0
- joint robotiq_85_left_inner_knuckle_joint: limit lower=-3.14 upper=3.14 effort=0.1 velocity=100.0 -> lower=-3.14 upper=3.14 effort=1000 velocity=1.0
- joint robotiq_85_right_finger_tip_joint: limit lower=-3.14 upper=3.14 effort=0.1 velocity=100.0 -> lower=-3.14 upper=3.14 effort=1000 velocity=1.0
- joint robotiq_85_right_inner_knuckle_joint: limit lower=-3.14 upper=3.14 effort=0.1 velocity=100.0 -> lower=-3.14 upper=3.14 effort=1000 velocity=1.0

Commit message: - robot mesh model path

File: assets/urdf/ur3_description/robot/ur3_robotiq85_gripper.urdf (robot description, URDF)
Before this commit: robot ur5, 21 links, 20 joints
Links:
- link base_link: geometry collision mesh filename=../meshes/collision/base.stl; visual mesh filename=../meshes/visual/base.dae
- link forearm_link: geometry collision mesh filename=../meshes/collision/forearm.stl; visual mesh filename=../meshes/visual/forearm.dae
- link robotiq_85_base_link: geometry collision mesh filename=../../robotiq_description/meshes/collision/robotiq_85_base_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; visual mesh filename=../../robotiq_description/meshes/visual/robotiq_85_base_lin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
- link robotiq_85_left_finger_link: geometry collision mesh filename=../../robotiq_description/meshes/collision/robotiq_85_finge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; visual mesh filename=../../robotiq_description/meshes/visual/robotiq_85_finger_l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
- link robotiq_85_left_finger_tip_link: geometry collision mesh filename=../../robotiq_description/meshes/collision/robotiq_85_finge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; visual mesh filename=../../robotiq_description/meshes/visual/robotiq_85_finger_t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
- link robotiq_85_left_inner_knuckle_link: geometry collision mesh filename=../../robotiq_description/meshes/collision/robotiq_85_inner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; visual mesh filename=../../robotiq_description/meshes/visual/robotiq_85_inner_kn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
- link robotiq_85_left_knuckle_link: geometry collision mesh filename=../../robotiq_description/meshes/collision/robotiq_85_knuck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; visual mesh filename=../../robotiq_description/meshes/visual/robotiq_85_knuckle_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
- link robotiq_85_right_finger_link: geometry collision mesh filename=../../robotiq_description/meshes/collision/robotiq_85_finge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; visual mesh filename=../../robotiq_description/meshes/visual/robotiq_85_finger_l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
- link robotiq_85_right_finger_tip_link: geometry collision mesh filename=../../robotiq_description/meshes/collision/robotiq_85_finge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; visual mesh filename=../../robotiq_description/meshes/visual/robotiq_85_finger_t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
- link robotiq_85_right_inner_knuckle_link: geometry collision mesh filename=../../robotiq_description/meshes/collision/robotiq_85_inner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; visual mesh filename=../../robotiq_description/meshes/visual/robotiq_85_inner_kn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
- link robotiq_85_right_knuckle_link: geometry collision mesh filename=../../robotiq_description/meshes/collision/robotiq_85_knuck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; visual mesh filename=../../robotiq_description/meshes/visual/robotiq_85_knuckle_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
- link robotiq_coupler: geometry collision mesh filename=../../robotiq_description/meshes/robotiq_85_coupler.stl; visual mesh filename=../../robotiq_description/meshes/robotiq_85_coupler.stl
- link shoulder_link: geometry collision mesh filename=../meshes/collision/shoulder.stl; visual mesh filename=../meshes/visual/shoulder.dae
- link upper_arm_link: geometry collision mesh filename=../meshes/collision/upperarm.stl; visual mesh filename=../meshes/visual/upperarm.dae
- link wrist_1_link: geometry collision mesh filename=../meshes/collision/wrist1.stl; visual mesh filename=../meshes/visual/wrist1.dae
- link wrist_2_link: geometry collision mesh filename=../meshes/collision/wrist2.stl; visual mesh filename=../meshes/visual/wrist2.dae
- link wrist_3_link: geometry collision mesh filename=../meshes/collision/wrist3.stl; visual mesh filename=../meshes/visual/wrist3.dae

Commit message: - robotiq_85 gripper urdf transformation error fixed - robotiq_85 coupler .dae file was added - dataset manager max frame tick is up to 30 - robot gui parsing function edit - pouring water skill sub-rewards - vr_test_main object selection - basis coordinate for alignment with real ur3

File: assets/urdf/ur3_description/robot/ur3_robotiq85_gripper.urdf (robot description, URDF)
Before this commit: robot ur5, 21 links, 20 joints
Links:
- link robotiq_coupler: geometry collision mesh filename=../../robotiq_description/meshes/robotiq_85_coupler.stl; visual mesh filename=../../robotiq_description/meshes/visual/robotiq_85_coupler.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
Joints:
- joint base_link-base_fixed_joint: origin xyz=0 0 0 rpy=0 0 -3.14159265359 -> xyz=0 0 0 rpy=0 0 0
- joint ee_fixed_joint: origin xyz=0.0 0.0819 0.0 rpy=0.0 0.0 1.57079632679 -> xyz=0.0 0.0819 0.0 rpy=-1.57079632679 0.0 0
- joint robotiq_85_base_joint: origin xyz=0 0 0.004 rpy=0 -1.57079632679 3.14159265359 -> xyz=0 0 0 rpy=0 0 -1.57079632679
- joint robotiq_coupler_joint: origin xyz=0 0 0.004 rpy=0 0 -1.57079632679 -> xyz=0 0 0 rpy=0 0 0
- joint wrist_3_link-tool0_fixed_joint: origin xyz=0 0.0819 0 rpy=-1.57079632679 0 0 -> xyz=0 0 0 rpy=-1.57079632679 0 0; parent wrist_3_link -> ee_link

Commit message: - matching coordinate system of base and tool between real UR3 and isaacgym's - update VR functions and module

File: assets/urdf/ur3_description/robot/ur3_robotiq85_gripper.urdf (robot description, URDF)
Before this commit: robot ur5, 21 links, 20 joints
Joints:
- joint robotiq_coupler_joint: origin xyz=0 0 0 rpy=0 0 0 -> xyz=0 0 0 rpy=-1.57079632679 0 0
- joint wrist_3_link-tool0_fixed_joint: origin xyz=0 0 0 rpy=-1.57079632679 0 0 -> xyz=0 0 0 rpy=0 0 0

Commit message: - ur3 urdf is fixed to correct the ee_link orientation - name, path, etc are fixed

File: assets/urdf/ur3_description/robot/ur3_robotiq85_gripper.urdf (robot description, URDF)
Before this commit: robot ur5, 21 links, 20 joints
Joints:
- joint ee_fixed_joint: origin xyz=0.0 0.0819 0.0 rpy=-1.57079632679 0.0 0 -> xyz=0.0 0.0819 0.0 rpy=-1.57079632679 3.14159265359 0

Commit message: - ur3-robotiq 2f-85 ee orientation fix

File: assets/urdf/ur3_description/robot/ur3_robotiq85_gripper.urdf (robot description, URDF)
Before this commit: robot ur5, 21 links, 20 joints
Joints:
- joint wrist_3_link-tool0_fixed_joint: origin xyz=0 0 0 rpy=0 0 0 -> xyz=0 0 0 rpy=0 0 3.14159265358
